File: AudioInjector.Octo.kicad_pcb (KiCad board)
At the start: 2 copper layers, 65 x 56.5 mm, 6 parts, among them P3 DAC_out, P4 ADC_in

Commit message: Latest updates for the template.
Connections:
- net /Codec/AGND renamed GND
- P3 pad 10: /Codec/AOUT6- -> (no net)
- P3 pad 11: /Codec/AOUT5- -> (no net)
- P3 pad 12: /Codec/AOUT6+ -> (no net)
- P3 pad 13: /Codec/AOUT3+ -> (no net)
- P3 pad 14: /Codec/AOUT4- -> (no net)
- P3 pad 15: /Codec/AOUT3- -> (no net)
- P3 pad 16: /Codec/AOUT4+ -> (no net)
- P3 pad 17: /Codec/AOUT1+ -> (no net)
- P3 pad 18: /Codec/AOUT2- -> (no net)
- P3 pad 19: /Codec/AOUT1- -> (no net)
- P3 pad 20: /Codec/AOUT2+ -> (no net)
- P3 pad 4: /Codec/MUTEC -> (no net)
- P3 pad 5: /Codec/AOUT7+ -> (no net)
- P3 pad 6: /Codec/AOUT8- -> (no net)
- P3 pad 7: /Codec/AOUT7- -> (no net)
- P3 pad 8: /Codec/AOUT8+ -> (no net)
- P3 pad 9: /Codec/AOUT5+ -> (no net)
- P4 pad 10: /Codec/ADC_fb3- -> (no net)
- P4 pad 12: /Codec/ADC_fb3+ -> (no net)
- P4 pad 14: /Codec/ADC_fb4- -> (no net)
- P4 pad 16: /Codec/ADC_fb4+ -> (no net)
- P4 pad 18: /Codec/ADC_fb5- -> (no net)
- P4 pad 2: /Codec/ADC_fb1- -> (no net)
- P4 pad 20: /Codec/ADC_fb5+ -> (no net)
- P4 pad 22: /Codec/ADC_fb6- -> (no net)
- P4 pad 24: /Codec/ADC_fb6+ -> (no net)
- P4 pad 4: /Codec/ADC_fb1+ -> (no net)
- P4 pad 6: /Codec/ADC_fb2- -> (no net)
- P4 pad 8: /Codec/ADC_fb2+ -> (no net)
